File: ControllerRP2040Scorpio/ControllerRP2040Scorpio.kicad_pcb (KiCad board)
At the start: 2 copper layers, 50.8 x 50.8 mm, 14 parts, among them J1 Conn_01x16_Socket, J2 Conn_01x12_Female, J3 Screw_Terminal_01x02, J4 Screw_Terminal_01x02, J5 Conn_01x02_Pin

Commit message: incremental updates
Routing:
- net +5V: track 68.8 -> 69.5 mm
Changed lines of the file:
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@@
 	)
 	(segment
-		(start 122.682 86.278323)
-		(end 140.384823 86.278323)
+		(start 131.998323 86.278323)
+		(end 137.1555 91.4355)
 		(width 2.54)
 		(layer "F.Cu")
@@
 	)
 	(segment
-		(start 113.538 102.616)
-		(end 113.538 86.36)
+		(start 108.433 86.36)
+		(end 115.062 86.36)
+		(width 2.54)
+		(layer "F.Cu")
+		(net 28)
+	)
+	(segment
+		(start 115.062 101.092)
+		(end 115.062 86.36)
+		(width 2.54)
+		(layer "F.Cu")
+		(net 28)
+	)
+	(segment
+		(start 115.062 86.36)
+		(end 122.600323 86.36)
 		(width 2.54)
 		(layer "F.Cu")
@@
 	)
 	(segment
-		(start 113.538 86.36)
-		(end 122.600323 86.36)
+		(start 122.682 86.278323)
+		(end 131.998323 86.278323)
+		(width 2.54)
+		(layer "F.Cu")
+		(net 28)
+	)
+	(segment
+		(start 137.1555 91.4355)
+		(end 145.542 91.4355)
 		(width 2.54)
 		(layer "F.Cu")
@@
 	(segment
 		(start 104.14 112.014)
-		(end 113.538 102.616)
+		(end 115.062 101.092)
 		(width 2.54)
 		(layer "F.Cu")
-		(net 28)
-	)
-	(segment
-		(start 108.433 86.36)
-		(end 113.538 86.36)
-		(width 2.54)
-		(layer "F.Cu")
-		(net 28)
-	)
-	(segment
-		(start 140.384823 86.278323)
-		(end 145.542 91.4355)
-		(width 2.54)
-		(layer "F.Cu")

Commit message: incremental updates
Parts:
- added REF**: KiCad-Logo2_6mm_SilkScreen, Symbol:KiCad-Logo2_6mm_SilkScreen, B.Cu at (127.0, 114.0)
- J1: footprint PinSocket_1x16_Feather:PinSocket_1x16_P2.54mm_Vertical -> MyFeatherPinSocket:PinSocket_1x16_P2.54mm_Vertical
- J2: footprint PinSocket_1x12_Feather:PinSocket_1x12_P2.54mm_Vertical -> MyFeatherPinSocket:PinSocket_1x12_P2.54mm_Vertical
- J3, J4: footprint Default:PHOENIX - TERM BLK 2P SIDE ENT 5.08MM PCB -> MyTerminalBlocks:PHOENIX - TERM BLK 2P SIDE ENT 5.08MM PCB

Commit message: incremental updates
Parts:
- removed C1: 1000uf, Capacitor_THT:CP_Radial_D10.0mm_P5.00mm
Routing:
- net +5V: track 69.1 -> 67.3 mm
Other:
- board text added: "Dripping Icicle Lights v1.0 Controller"
- board text removed: "Dripping Icicle Lights Controller v1.0"
