File: ControllerRP2040Scorpio/ControllerRP2040Scorpio.kicad_sch (KiCad schematic)
At the start: 6 parts, among them J1 Conn_01x16_Socket, J2 Conn_01x12_Female, J3 Screw_Terminal_01x02, J4 Screw_Terminal_01x02, J5 Conn_01x02_Pin

Commit message: incremental updates
Parts:
- C1: DigiKey Part https://www.digikey.com/en/products/detail/rubycon/25PX1000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 -> 1189-1583-1-ND
- J1: footprint PinSocket_1x16_Feather:PinSocket_1x16_P2.54mm_Vertical -> MyFeatherPinSocket:PinSocket_1x16_P2.54mm_Vertical
- J2: footprint PinSocket_1x12_Feather:PinSocket_1x12_P2.54mm_Vertical -> MyFeatherPinSocket:PinSocket_1x12_P2.54mm_Vertical
- J3, J4: footprint Default:PHOENIX - TERM BLK 2P SIDE ENT 5.08MM PCB -> MyTerminalBlocks:PHOENIX - TERM BLK 2P SIDE ENT 5.08MM PCB
Changed lines of the file:
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@@
 			)
 		)
-		(property "DigiKey Part" "https://www.digikey.com/en/products/detail/rubycon/25PX1000MEFCT810X16/3134863"
+		(property "DigiKey Part" "1189-1583-1-ND"
 			(at 109.22 123.19 0)
 			(effects
@@
 			)
 		)
-		(property "Footprint" "Default:PHOENIX - TERM BLK 2P SIDE ENT 5.08MM PCB"
+		(property "Footprint" "MyTerminalBlocks:PHOENIX - TERM BLK 2P SIDE ENT 5.08MM PCB"
 			(at 119.38 104.14 0)
 			(effects
@@
 			)
 		)
-		(property "Footprint" "PinSocket_1x16_Feather:PinSocket_1x16_P2.54mm_Vertical"
+		(property "Footprint" "MyFeatherPinSocket:PinSocket_1x16_P2.54mm_Vertical"
 			(at 153.67 106.68 0)
 			(effects
@@
 			)
 		)
-		(property "Footprint" "Default:PHOENIX - TERM BLK 2P SIDE ENT 5.08MM PCB"
+		(property "Footprint" "MyTerminalBlocks:PHOENIX - TERM BLK 2P SIDE ENT 5.08MM PCB"
 			(at 185.42 107.95 0)
 			(effects
@@
 			)
 		)
-		(property "Datasheet" "~"
+		(property "Datasheet" "https://www.phoenixcontact.com/product/pdf/api/v1/MTcyOTEyOA?_realm=us&_locale=en-US&blocks=commercial-data%2Ctechnical-data%2Cdrawings%2Capprovals%2Cclassifications%2Cenvironmental-compliance-data%2Call-accessories"
 			(at 185.42 107.95 0)
 			(effects
@@
 			)
 		)
-		(property "Footprint" "PinSocket_1x12_Feather:PinSocket_1x12_P2.54mm_Vertical"
+		(property "Footprint" "MyFeatherPinSocket:PinSocket_1x12_P2.54mm_Vertical"
 			(at 157.48 111.76 0)
 			(effects

Commit message: incremental updates
Parts:
- removed C1: 1000uf, Capacitor_THT:CP_Radial_D10.0mm_P5.00mm, symbol Device:C_Polarized_US
Other:
- moved on the sheet: J3
