File: LedStrandPower/LedStrandPower.kicad_pcb (KiCad board)
At the start: 2 copper layers, 55.9 x 25.4 mm, 9 parts, among them J1 PJ-102B, J2 Conn_01x01_Pin, J3 Screw_Terminal_01x03, J4 Screw_Terminal_01x02

Commit message: incremental updates
Parts:
- added C1: 1000uf, Capacitor_THT:CP_Radial_D10.0mm_P5.00mm, F.Cu at (132.2, 95.2)
- moved J2 28.8 mm to (132.8, 107.3)
- moved J3 22.0 mm to (148.6, 111.4)
- moved J4 11.0 mm to (136.4, 111.4)
- moved REF** 10.2 mm to (152.4, 97.8)
Routing:
- net +5V: track 48.9 -> 55.0 mm
- net /Data: track 29.3 -> 25.9 mm
Other:
- board text added: "Dripping Icicle Lights v1.0 Power & Splat Strip"
- board text added: "Splat"
- board text removed: "Dripping Icicle Lights v1.0 Splat Strip"
