File: LedStrandDrip/LedStrandDrip.kicad_pcb (KiCad board)
At the start: 2 copper layers, 40.6 x 20.3 mm, 9 parts, among them J1 Screw_Terminal_01x02, J2 Conn_01x01_Pin, J3 Screw_Terminal_01x03, J4 Screw_Terminal_01x02

Commit message: incremetal updates
Routing:
- net +5V: track 37.2 -> 34.0 mm
Other:
- board text added: "Data In"
- board text added: "Drip Strand"
- board text added: "Dripping Icicle Lights v1.0 Drip Strand"
- board text removed: "Data Out"
Changed lines of the file:
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@@
 		(layer "User.1")
+	)
+	(gr_text "Dripping Icicle Lights v1.0\nDrip Strand"
+		(at 152.4 94.615 0)
+		(layer "B.SilkS")
+		(effects
+			(font
+				(size 1 1)
+				(thickness 0.1)
+			)
+			(justify mirror)
+		)
 	)
 	(gr_text "https://github.com/ngdrascal/IcicleLights"
@@
 		)
 	)
+	(gr_text "Drip Strand"
+		(at 155.448 106.68 0)
+		(layer "F.SilkS")
+		(effects
+			(font
+				(size 1 1)
+				(thickness 0.1)
+			)
+		)
+	)
 	(gr_text "GND"
 		(at 147.32 92.71 180)
@@
 		)
 	)
-	(gr_text "Data\nOut"
-		(at 147.32 109.855 0)
+	(gr_text "Data In"
+		(at 147.32 109.22 0)
 		(layer "F.SilkS")
 		(effects
@@
 	)
 	(segment
-		(start 154.94 93.345)
-		(end 141.605 93.345)
+		(start 154.446 94.996)
+		(end 157.48 98.03)
 		(width 2.54)
 		(layer "F.Cu")
@@
 	)
 	(segment
-		(start 138.67 96.28)
-		(end 138.67 99.06)
+		(start 140.97 94.996)
+		(end 154.446 94.996)
 		(width 2.54)
 		(layer "F.Cu")
@@
 	)
 	(segment
-		(start 157.48 95.885)
-		(end 154.94 93.345)
+		(start 138.67 97.296)
+		(end 140.97 94.996)
 		(width 2.54)
 		(layer "F.Cu")
@@
 	)
 	(segment
-		(start 141.605 93.345)
-		(end 138.67 96.28)
+		(start 138.67 99.06)
+		(end 138.67 97.296)
 		(width 2.54)
 		(layer "F.Cu")
-		(net 2)
-	)
-	(segment
-		(start 157.48 98.03)
-		(end 157.48 95.885)
-		(width 2.54)
-		(layer "F.Cu")
