File: LedStrandSplat/LedStrandSplat.kicad_pcb (KiCad board)
At the start: 2 copper layers, 55.9 x 25.4 mm, 10 parts, among them J1 PJ-102B, J2 Conn_01x01_Pin, J3 Screw_Terminal_01x03, J4 Screw_Terminal_01x02

Commit message: incremetal updates
Parts:
- moved J2 2.92 mm to (132.8, 110.2)
Routing:
- net /Data: track 25.9 -> 24.6 mm
Other:
- board text added: "Dripping Icicle Lights v1.0 Splat Strand"
- board text removed: "Dripping Icicle Lights v1.0 Power & Splat Strip"
- board text removed: "Splat"
Changed lines of the file:
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@@
 	(footprint "Connector_PinHeader_2.54mm:PinHeader_1x01_P2.54mm_Vertical"
 		(layer "F.Cu")
-		(at 132.842 107.315 180)
+		(at 132.842 110.236 180)
 		(descr "Through hole straight pin header, 1x01, 2.54mm pitch, single row")
 		(tags "Through hole pin header THT 1x01 2.54mm single row")
@@
 		)
 	)
-	(gr_text "Splat"
-		(at 132.842 111.125 0)
+	(gr_text "Controller"
+		(at 138.8745 101.6 0)
 		(layer "F.SilkS")
 		(effects
@@
 		)
 	)
-	(gr_text "Controller"
-		(at 138.8745 101.6 0)
+	(gr_text "Data"
+		(at 154.305 113.03 0)
 		(layer "F.SilkS")
 		(effects
@@
 				(thickness 0.1)
 			)
-		)
-	)
-	(gr_text "Data"
-		(at 154.305 113.03 0)
+			(justify left)
+		)
+	)
+	(gr_text "GND"
+		(at 144.272 113.03 0)
 		(layer "F.SilkS")
 		(effects
@@
 				(thickness 0.1)
 			)
-			(justify left)
-		)
-	)
-	(gr_text "GND"
-		(at 144.272 113.03 0)
+		)
+	)
+	(gr_text "5V Power"
+		(at 170.18 97.917 0)
 		(layer "F.SilkS")
 		(effects
@@
 		)
 	)
-	(gr_text "5V Power"
-		(at 170.18 97.917 0)
+	(gr_text "+5"
+		(at 151.13 113.03 0)
 		(layer "F.SilkS")
 		(effects
@@
 		)
 	)
-	(gr_text "+5"
-		(at 151.13 113.03 0)
+	(gr_text "GND"
+		(at 161.29 113.03 0)
 		(layer "F.SilkS")
 		(effects
@@
 		)
 	)
-	(gr_text "GND"
-		(at 161.29 113.03 0)
+	(gr_text "Dripping Icicle Lights v1.0\nSplat Strand"
+		(at 152.4 92.075 0)
 		(layer "F.SilkS")
 		(effects
@@
 		)
 	)
-	(gr_text "Dripping Icicle Lights v1.0\nPower & Splat Strip"
-		(at 152.4 92.075 0)
+	(gr_text "Data In"
+		(at 132.842 113.03 0)
 		(layer "F.SilkS")
 		(effects
@@
 		)
 	)
-	(gr_text "Data In"
-		(at 132.842 113.03 0)
+	(gr_text "Splat Strip"
+		(at 156.21 101.6 0)
 		(layer "F.SilkS")
 		(effects
@@
 		)
 	)
-	(gr_text "Splat Strip"
-		(at 156.21 101.6 0)
-		(layer "F.SilkS")
-		(effects
-			(font
-				(size 1 1)
-				(thickness 0.1)
-			)
-		)
-	)
 	(segment
-		(start 135.636 110.236)
+		(start 156.21 107.315)
 		(end 153.289 110.236)
 		(width 0.2)
@@
 	)
 	(segment
-		(start 132.842 107.315)
-		(end 135.636 110.109)
+		(start 153.289 110.236)
+		(end 132.842 110.236)
 		(width 0.2)
 		(layer "F.Cu")
-		(net 1)
-	)
-	(segment
-		(start 153.289 110.236)
-		(end 156.21 107.315)
-		(width 0.2)
-		(layer "F.Cu")
-		(net 1)
-	)
-	(segment
-		(start 135.636 110.109)
-		(end 135.636 110.236)
-		(width 0.2)
-		(layer "F.Cu")
