File: LedSplatStrand/LedSplatStrand.kicad_sch (KiCad schematic)
At the start: 5 parts, among them J1 PJ-102B, J2 Conn_01x01_Pin, J3 Screw_Terminal_01x03, J4 Screw_Terminal_01x02

Commit message: incremental updates
Other:
- moved on the sheet: J3, J4
Changed lines of the file:
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@@
 	(wire
 		(pts
-			(xy 152.4 90.17) (xy 152.4 91.44)
-		)
-		(stroke
-			(width 0)
-			(type default)
-		)
-	)
-	(wire
-		(pts
-			(xy 149.86 93.98) (xy 153.67 93.98)
-		)
-		(stroke
-			(width 0)
-			(type default)
-		)
-	)
-	(wire
-		(pts
-			(xy 152.4 110.49) (xy 152.4 111.76)
-		)
-		(stroke
-			(width 0)
-			(type default)
-		)
-	)
-	(wire
-		(pts
-			(xy 143.51 96.52) (xy 153.67 96.52)
-		)
-		(stroke
-			(width 0)
-			(type default)
-		)
-	)
-	(wire
-		(pts
-			(xy 152.4 106.68) (xy 152.4 107.95)
+			(xy 133.35 77.47) (xy 133.35 78.74)
+		)
+		(stroke
+			(width 0)
+			(type default)
+		)
+	)
+	(wire
+		(pts
+			(xy 130.81 81.28) (xy 134.62 81.28)
+		)
+		(stroke
+			(width 0)
+			(type default)
+		)
+	)
+	(wire
+		(pts
+			(xy 151.13 93.98) (xy 151.13 95.25)
+		)
+		(stroke
+			(width 0)
+			(type default)
+		)
+	)
+	(wire
+		(pts
+			(xy 133.35 83.82) (xy 134.62 83.82)
+		)
+		(stroke
+			(width 0)
+			(type default)
+		)
+	)
+	(wire
+		(pts
+			(xy 151.13 90.17) (xy 151.13 91.44)
 		)
 		(stroke
@@
 	(wire
 		(pts
-			(xy 153.67 110.49) (xy 152.4 110.49)
+			(xy 152.4 93.98) (xy 151.13 93.98)
 		)
 		(stroke
@@
 	(wire
 		(pts
-			(xy 152.4 91.44) (xy 153.67 91.44)
-		)
-		(stroke
-			(width 0)
-			(type default)
-		)
-	)
-	(wire
-		(pts
-			(xy 152.4 107.95) (xy 153.67 107.95)
+			(xy 133.35 78.74) (xy 134.62 78.74)
+		)
+		(stroke
+			(width 0)
+			(type default)
+		)
+	)
+	(wire
+		(pts
+			(xy 151.13 91.44) (xy 152.4 91.44)
 		)
 		(stroke
@@
 	(wire
 		(pts
-			(xy 143.51 96.52) (xy 143.51 97.79)
+			(xy 133.35 83.82) (xy 133.35 85.09)
 		)
 		(stroke
@@
 	)
 	(label "Data"
-		(at 149.86 93.98 0)
+		(at 130.81 81.28 0)
 		(fields_autoplaced yes)
 		(effects
@@
 	(symbol
 		(lib_id "power:GND")
-		(at 152.4 111.76 0)
+		(at 151.13 95.25 0)
 		(unit 1)
 		(exclude_from_sim no)
@@
 		(dnp no)
 		(property "Reference" "#PWR06"
-			(at 152.4 118.11 0)
+			(at 151.13 101.6 0)
 			(effects
 				(font
@@
 		)
 		(property "Value" "GND"
-			(at 152.4 115.57 0)
+			(at 151.13 99.06 0)
 			(effects
 				(font
@@
 		)
 		(property "Footprint" ""
-			(at 152.4 111.76 0)
+			(at 151.13 95.25 0)
 			(effects
 				(font
@@
 		)
 		(property "Datasheet" ""
-			(at 152.4 111.76 0)
+			(at 151.13 95.25 0)
 			(effects
 				(font
@@
 		)
 		(property "Description" "Power symbol creates a global label with name \"GND\" , ground"
-			(at 152.4 111.76 0)
+			(at 151.13 95.25 0)
 			(effects
 				(font
@@
 	(symbol
 		(lib_id "Connector:Screw_Terminal_01x02")
-		(at 158.75 107.95 0)
+		(at 157.48 91.44 0)
 		(unit 1)
 		(exclude_from_sim no)
@@
 		(dnp no)
 		(property "Reference" "J4"
-			(at 157.734 105.41 0)
+			(at 156.464 88.9 0)
 			(effects
 				(font
@@
 		)
 		(property "Value" "Screw_Terminal_01x02"
-			(at 147.828 117.856 0)
+			(at 146.558 101.346 0)
 			(effects
 				(font
@@
 		)
 		(property "Footprint" "MyTerminalBlock:PHOENIX - TERM BLK 2P SIDE ENT 5.08MM PCB"
-			(at 158.75 107.95 0)
+			(at 157.48 91.44 0)
 			(effects
 				(font
@@
 		)
 		(property "Datasheet" "~"
-			(at 158.75 107.95 0)
+			(at 157.48 91.44 0)
 			(effects
 				(font
@@
 		)
 		(property "Description" "Generic screw terminal, single row, 01x02, script generated (kicad-library-utils/schlib/autogen/connector/)"
-			(at 158.75 107.95 0)
+			(at 157.48 91.44 0)
 			(effects
 				(font
@@
 		)
 		(property "DigiKey Part" "277-1247-ND"
-			(at 158.75 107.95 0)
+			(at 157.48 91.44 0)
 			(effects
 				(font
@@
 	(symbol
 		(lib_id "power:+5V")
-		(at 152.4 90.17 0)
+		(at 133.35 77.47 0)
 		(unit 1)
 		(exclude_from_sim no)
@@
 		(dnp no)
 		(property "Reference" "#PWR07"
-			(at 152.4 93.98 0)
+			(at 133.35 81.28 0)
 			(effects
 				(font
@@
 		)
 		(property "Value" "+5V"
-			(at 152.146 86.36 0)
+			(at 133.096 73.66 0)
 			(effects
 				(font
@@
 		)
 		(property "Footprint" ""
-			(at 152.4 90.17 0)
+			(at 133.35 77.47 0)
 			(effects
 				(font
@@
 		)
 		(property "Datasheet" ""
-			(at 152.4 90.17 0)
+			(at 133.35 77.47 0)
 			(effects
 				(font
@@
 		)
 		(property "Description" "Power symbol creates a global label with name \"+5V\""
-			(at 152.4 90.17 0)
+			(at 133.35 77.47 0)
 			(effects
 				(font
@@
 	(symbol
 		(lib_id "Connector:Screw_Terminal_01x03")
-		(at 158.75 93.98 0)
+		(at 139.7 81.28 0)
 		(unit 1)
 		(exclude_from_sim no)
@@
 		(dnp no)
 		(property "Reference" "J3"
-			(at 157.48 89.154 0)
+			(at 138.43 76.454 0)
 			(effects
 				(font
@@
 		)
 		(property "Value" "Screw_Terminal_01x03"
-			(at 148.59 99.06 0)
+			(at 129.54 86.36 0)
 			(effects
 				(font
@@
 		)
 		(property "Footprint" "MyTerminalBlock:PHOENIX - TERM BLK 3P SIDE ENT 5.08MM PCB"
-			(at 158.75 93.98 0)
+			(at 139.7 81.28 0)
 			(effects
 				(font
@@
 		)
 		(property "Datasheet" "~"
-			(at 158.75 93.98 0)
+			(at 139.7 81.28 0)
 			(effects
 				(font
@@
 		)
 		(property "Description" "Generic screw terminal, single row, 01x03, script generated (kicad-library-utils/schlib/autogen/connector/)"
-			(at 158.75 93.98 0)
+			(at 139.7 81.28 0)
 			(effects
 				(font
@@
 		)
 		(property "DigiKey Part" "277-1248-ND"
-			(at 158.75 93.98 0)
+			(at 139.7 81.28 0)
 			(effects
 				(font
@@
 	(symbol
 		(lib_id "power:+5V")
-		(at 152.4 106.68 0)
+		(at 151.13 90.17 0)
 		(unit 1)
 		(exclude_from_sim no)
@@
 		(dnp no)
 		(property "Reference" "#PWR05"
-			(at 152.4 110.49 0)
+			(at 151.13 93.98 0)
 			(effects
 				(font
@@
 		)
 		(property "Value" "+5V"
-			(at 152.146 102.87 0)
+			(at 150.876 86.36 0)
 			(effects
 				(font
@@
 		)
 		(property "Footprint" ""
-			(at 152.4 106.68 0)
+			(at 151.13 90.17 0)
 			(effects
 				(font
@@
 		)
 		(property "Datasheet" ""
-			(at 152.4 106.68 0)
+			(at 151.13 90.17 0)
 			(effects
 				(font
@@
 		)
 		(property "Description" "Power symbol creates a global label with name \"+5V\""
-			(at 152.4 106.68 0)
+			(at 151.13 90.17 0)
 			(effects
 				(font
@@
 	(symbol
 		(lib_id "power:GND")
-		(at 143.51 97.79 0)
+		(at 133.35 85.09 0)
 		(unit 1)
 		(exclude_from_sim no)
@@
 		(dnp no)
 		(property "Reference" "#PWR08"
-			(at 143.51 104.14 0)
+			(at 133.35 91.44 0)
 			(effects
 				(font
@@
 		)
 		(property "Value" "GND"
-			(at 143.51 101.6 0)
+			(at 133.35 88.9 0)
 			(effects
 				(font
@@
 		)
 		(property "Footprint" ""
-			(at 143.51 97.79 0)
+			(at 133.35 85.09 0)
 			(effects
 				(font
@@
 		)
 		(property "Datasheet" ""
-			(at 143.51 97.79 0)
+			(at 133.35 85.09 0)
 			(effects
 				(font
@@
 		)
 		(property "Description" "Power symbol creates a global label with name \"GND\" , ground"
-			(at 143.51 97.79 0)
-			(effects
-				(font
+			(at 133.35 85.09 0)
+			(effects
+				(font
