File: LedController/LedController.kicad_pcb (KiCad board)
At the start: 2 copper layers, 50.8 x 50.8 mm, 14 parts, among them J1 Conn_01x16_Socket, J2 Conn_01x12_Female, J3 Screw_Terminal_01x02, J4 Screw_Terminal_01x02, J5 Conn_01x02_Pin

Commit message: incremental updates
Parts:
- added J6: Conn_01x01_Pin, Connector_PinHeader_2.54mm:PinHeader_1x01_P2.54mm_Vertical, F.Cu at (127.0, 90.7)
- added J7: Screw_Terminal_01x03, MyTerminalBlocks:PHOENIX - TERM BLK 3P SIDE ENT 5.08MM PCB, F.Cu at (119.4, 86.9)
- moved J4 12.8 mm to (141.7, 83.8), turned to -90 degrees
- moved J3 0.24 mm to (104.1, 83.8)
Routing:
- net /Data: track 0.00 -> 7.87 mm
- net +5V: track 67.3 -> 70.2 mm
Other:
- board text added: "+5"
- board text added: "Data"
- board text added: "Data In"

Commit message: incremental updates
Parts:
- moved J7 17.3 mm to (134.6, 78.8), turned to 180 degrees
Changed lines of the file:
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@@
 	(footprint "MyTerminalBlocks:PHOENIX - TERM BLK 3P SIDE ENT 5.08MM PCB"
 		(layer "F.Cu")
-		(at 119.38 86.854)
+		(at 134.62 78.754 180)
 		(property "Reference" "J7"
-			(at 3.175 -9.135 0)
+			(at 3.175 -9.135 360)
 			(layer "F.SilkS")
 			(hide yes)
@@
 		)
 		(property "Value" "Screw_Terminal_01x03"
-			(at 9.525 1.115 0)
+			(at 9.525 1.115 360)
 			(layer "F.Fab")
 			(hide yes)
@@
 		)
 		(property "Footprint" "MyTerminalBlocks:PHOENIX - TERM BLK 3P SIDE ENT 5.08MM PCB"
-			(at 0 0 0)
+			(at 0 0 360)
 			(layer "F.Fab")
 			(hide yes)
@@
 		)
 		(property "Datasheet" ""
-			(at 0 0 0)
+			(at 0 0 360)
 			(layer "F.Fab")
 			(hide yes)
@@
 		)
 		(property "Description" "Generic screw terminal, single row, 01x03, script generated (kicad-library-utils/schlib/autogen/connector/)"
-			(at 0 0 0)
+			(at 0 0 360)
 			(layer "F.Fab")
 			(hide yes)
@@
 		)
 		(property "DigiKey Part" "277-1248-ND"
-			(at 0 0 0)
+			(at 0 0 180)
 			(unlocked yes)
 			(layer "F.Fab")
@@
 		(attr through_hole)
 		(fp_line
-			(start 0 -8.15)
-			(end 0 0)
+			(start 15.24 0)
+			(end 15.24 -8.15)
 			(stroke
 				(width 0.127)
@@
 		)
 		(fp_line
-			(start 0 0)
-			(end 15.24 0)
+			(start 15.24 -8.15)
+			(end 0 -8.15)
 			(stroke
 				(width 0.127)
@@
 		)
 		(fp_line
-			(start 15.24 -8.15)
-			(end 0 -8.15)
+			(start 0 0)
+			(end 15.24 0)
 			(stroke
 				(width 0.127)
@@
 		)
 		(fp_line
-			(start 15.24 0)
-			(end 15.24 -8.15)
+			(start 0 -8.15)
+			(end 0 0)
 			(stroke
 				(width 0.127)
@@
 		)
 		(fp_line
-			(start -0.82 -8.4)
-			(end -0.82 0.25)
+			(start 15.49 0.25)
+			(end 15.49 -8.4)
 			(stroke
 				(width 0.05)
@@
 		)
 		(fp_line
-			(start -0.82 0.25)
-			(end 15.49 0.25)
+			(start 15.49 -8.4)
+			(end -0.82 -8.4)
 			(stroke
 				(width 0.05)
@@
 		)
 		(fp_line
-			(start 15.49 -8.4)
-			(end -0.82 -8.4)
+			(start -0.82 0.25)
+			(end 15.49 0.25)
 			(stroke
 				(width 0.05)
@@
 		)
 		(fp_line
-			(start 15.49 0.25)
-			(end 15.49 -8.4)
+			(start -0.82 -8.4)
+			(end -0.82 0.25)
 			(stroke
 				(width 0.05)
@@
 		)
 		(fp_line
-			(start 0 -8.15)
-			(end 0 0)
+			(start 15.24 0)
+			(end 15.24 -8.15)
 			(stroke
 				(width 0.127)
@@
 		)
 		(fp_line
-			(start 0 0)
-			(end 15.24 0)
+			(start 15.24 -8.15)
+			(end 0 -8.15)
 			(stroke
 				(width 0.127)
@@
 		)
 		(fp_line
-			(start 15.24 -8.15)
-			(end 0 -8.15)
+			(start 0 0)
+			(end 15.24 0)
 			(stroke
 				(width 0.127)
@@
 		)
 		(fp_line
-			(start 15.24 0)
-			(end 15.24 -8.15)
+			(start 0 -8.15)
+			(end 0 0)
 			(stroke
 				(width 0.127)
@@
 		)
 		(pad "1" thru_hole rect
-			(at 2.54 -4.05)
+			(at 2.54 -4.05 180)
 			(size 1.95 1.95)
 			(drill 1.3)
@@
 		)
 		(pad "2" thru_hole circle
-			(at 7.62 -4.05)
+			(at 7.62 -4.05 180)
 			(size 1.95 1.95)
 			(drill 1.3)
@@
 		)
 		(pad "3" thru_hole circle
-			(at 12.7 -4.05)
+			(at 12.7 -4.05 180)
 			(size 1.95 1.95)
 			(drill 1.3)
@@
 	)
 	(gr_text "+5V"
-		(at 151.638 93.218 90)
+		(at 151.638 88.138 90)
 		(layer "F.SilkS")
 		(effects
@@
 	)
 	(gr_text "GND"
-		(at 151.638 88.138 90)
+		(at 151.638 93.218 90)
 		(layer "F.SilkS")
 		(effects
@@
 	)
 	(segment
-		(start 121.92 86.36)
-		(end 145.796 86.36)
+		(start 132.08 82.804)
+		(end 132.08 86.36)
 		(width 2.54)
 		(layer "F.Cu")
@@
 	)
 	(segment
-		(start 104.14 112.014)
-		(end 112.268 103.886)
+		(start 132.08 86.36)
+		(end 145.796 86.36)
 		(width 2.54)
 		(layer "F.Cu")
@@
 	)
 	(segment
-		(start 112.268 103.886)
-		(end 112.268 86.36)
+		(start 121.92 86.36)
+		(end 132.08 86.36)
 		(width 2.54)
 		(layer "F.Cu")
@@
 	)
 	(segment
-		(start 121.92 82.804)
-		(end 121.92 86.36)
+		(start 104.14 112.014)
+		(end 112.268 103.886)
+		(width 2.54)
+		(layer "F.Cu")
+		(net 28)
+	)
+	(segment
+		(start 112.268 103.886)
+		(end 112.268 86.36)
 		(width 2.54)
 		(layer "F.Cu")

Commit message: incremental updates
Parts:
- moved J4 13.0 mm to (149.8, 94.0), turned to 90 degrees
Connections:
- J4 pad 1: +5V -> GND
- J4 pad 2: GND -> +5V
Changed lines of the file:
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@@
 		(at 134.62 78.754 180)
 		(property "Reference" "J7"
-			(at 3.175 -9.135 360)
+			(at 3.175 -9.135 0)
 			(layer "F.SilkS")
 			(hide yes)
@@
 		)
 		(property "Value" "Screw_Terminal_01x03"
-			(at 9.525 1.115 360)
+			(at 9.525 1.115 0)
 			(layer "F.Fab")
 			(hide yes)
@@
 		)
 		(property "Footprint" "MyTerminalBlocks:PHOENIX - TERM BLK 3P SIDE ENT 5.08MM PCB"
-			(at 0 0 360)
+			(at 0 0 0)
 			(layer "F.Fab")
 			(hide yes)
@@
 		)
 		(property "Datasheet" ""
-			(at 0 0 360)
+			(at 0 0 0)
 			(layer "F.Fab")
 			(hide yes)
@@
 		)
 		(property "Description" "Generic screw terminal, single row, 01x03, script generated (kicad-library-utils/schlib/autogen/connector/)"
-			(at 0 0 360)
+			(at 0 0 0)
 			(layer "F.Fab")
 			(hide yes)
@@
 	(footprint "MyTerminalBlocks:PHOENIX - TERM BLK 2P SIDE ENT 5.08MM PCB"
 		(layer "F.Cu")
-		(at 141.746 83.82 -90)
+		(at 149.846 93.98 90)
 		(property "Reference" "J4"
 			(at 5.3295 -9.135 90)
@@
 		)
 		(property "DigiKey Part" "277-1247-ND"
-			(at 0 0 -90)
+			(at 0 0 90)
 			(unlocked yes)
 			(layer "F.Fab")
@@
 		(attr through_hole)
 		(fp_line
-			(start 0 0)
-			(end 10.16 0)
+			(start 10.16 -8.15)
+			(end 0 -8.15)
 			(stroke
 				(width 0.127)
@@
 		)
 		(fp_line
-			(start 10.16 0)
-			(end 10.16 -8.15)
+			(start 0 -8.15)
+			(end 0 0)
 			(stroke
 				(width 0.127)
@@
 		)
 		(fp_line
-			(start 0 -8.15)
-			(end 0 0)
+			(start 10.16 0)
+			(end 10.16 -8.15)
 			(stroke
 				(width 0.127)
@@
 		)
 		(fp_line
-			(start 10.16 -8.15)
-			(end 0 -8.15)
+			(start 0 0)
+			(end 10.16 0)
 			(stroke
 				(width 0.127)
@@
 		)
 		(fp_line
-			(start -0.82 0.25)
-			(end 10.41 0.25)
+			(start 10.41 -8.4)
+			(end -0.82 -8.4)
 			(stroke
 				(width 0.05)
@@
 		)
 		(fp_line
-			(start 10.41 0.25)
-			(end 10.41 -8.4)
+			(start -0.82 -8.4)
+			(end -0.82 0.25)
 			(stroke
 				(width 0.05)
@@
 		)
 		(fp_line
-			(start -0.82 -8.4)
-			(end -0.82 0.25)
+			(start 10.41 0.25)
+			(end 10.41 -8.4)
 			(stroke
 				(width 0.05)
@@
 		)
 		(fp_line
-			(start 10.41 -8.4)
-			(end -0.82 -8.4)
+			(start -0.82 0.25)
+			(end 10.41 0.25)
 			(stroke
 				(width 0.05)
@@
 		)
 		(fp_line
-			(start 0 0)
-			(end 10.16 0)
+			(start 10.16 -8.15)
+			(end 0 -8.15)
 			(stroke
 				(width 0.127)
@@
 		)
 		(fp_line
-			(start 10.16 0)
-			(end 10.16 -8.15)
+			(start 0 -8.15)
+			(end 0 0)
 			(stroke
 				(width 0.127)
@@
 		)
 		(fp_line
-			(start 0 -8.15)
-			(end 0 0)
+			(start 10.16 0)
+			(end 10.16 -8.15)
 			(stroke
 				(width 0.127)
@@
 		)
 		(fp_line
-			(start 10.16 -8.15)
-			(end 0 -8.15)
+			(start 0 0)
+			(end 10.16 0)
 			(stroke
 				(width 0.127)
@@
 		)
 		(pad "1" thru_hole rect
-			(at 2.54 -4.05 270)
+			(at 2.54 -4.05 90)
 			(size 1.95 1.95)
 			(drill 1.3)
 			(layers "*.Cu" "*.Mask")
 			(remove_unused_layers no)
-			(net 28 "+5V")
+			(net 13 "GND")
 			(pinfunction "Pin_1")
 			(pintype "passive")
@@
 		)
 		(pad "2" thru_hole circle
-			(at 7.62 -4.05 270)
+			(at 7.62 -4.05 90)
 			(size 1.95 1.95)
 			(drill 1.3)
 			(layers "*.Cu" "*.Mask")
 			(remove_unused_layers no)
-			(net 13 "GND")
+			(net 28 "+5V")
 			(pinfunction "Pin_2")
 			(pintype "passive")
@@
 	)
 	(segment
-		(start 132.08 86.36)
-		(end 145.796 86.36)
-		(width 2.54)
-		(layer "F.Cu")
-		(net 28)
-	)
-	(segment
 		(start 121.92 86.36)
 		(end 132.08 86.36)
@@
 		(width 2.54)
 		(layer "F.Cu")
+		(net 28)
+	)
+	(segment
+		(start 145.796 86.36)
+		(end 132.08 86.36)
+		(width 2.54)
+		(layer "F.Cu")
