File: LedController/LedController.kicad_sch (KiCad schematic)
At the start: 5 parts, among them J1 Conn_01x16_Socket, J2 Conn_01x12_Female, J3 Screw_Terminal_01x02, J4 Screw_Terminal_01x02, J5 Conn_01x02_Pin

Commit message: incremental updates
Parts:
- added J6: Conn_01x01_Pin, Connector_PinHeader_2.54mm:PinHeader_1x01_P2.54mm_Vertical, symbol Connector:Conn_01x01_Pin
- added J7: Screw_Terminal_01x03, MyTerminalBlocks:PHOENIX - TERM BLK 3P SIDE ENT 5.08MM PCB, symbol Connector:Screw_Terminal_01x03
Connections:
- net +5V: now also J7.1 (Pin_1)
- net GND: now also J7.3 (Pin_3)
- new net Data: J6.1 (Pin_1), J7.2 (Pin_2)

Commit message: incremental updates
Connections:
- net +5V: now also J4.2 (Pin_2); no longer J4.1 (Pin_1)
- net GND: now also J4.1 (Pin_1); no longer J4.2 (Pin_2)
Other:
- moved on the sheet: J4
Changed lines of the file:
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@@
-	(wire
-		(pts
-			(xy 179.07 106.68) (xy 179.07 107.95)
-		)
-		(stroke
-			(width 0)
-			(type default)
-		)
-	)
 	(wire
 		(pts
@@
 	(wire
 		(pts
+			(xy 191.77 107.95) (xy 191.77 109.22)
+		)
+		(stroke
+			(width 0)
+			(type default)
+		)
+	)
+	(wire
+		(pts
 			(xy 142.24 119.38) (xy 148.59 119.38)
 		)
@@
 	(wire
 		(pts
-			(xy 179.07 107.95) (xy 180.34 107.95)
-		)
-		(stroke
-			(width 0)
-			(type default)
-		)
-	)
-	(wire
-		(pts
 			(xy 162.56 101.6) (xy 168.91 101.6)
 		)
@@
 	(wire
 		(pts
+			(xy 190.5 105.41) (xy 191.77 105.41)
+		)
+		(stroke
+			(width 0)
+			(type default)
+		)
+	)
+	(wire
+		(pts
 			(xy 142.24 104.14) (xy 148.59 104.14)
 		)
@@
 	(wire
 		(pts
-			(xy 179.07 111.76) (xy 179.07 110.49)
-		)
-		(stroke
-			(width 0)
-			(type default)
-		)
-	)
-	(wire
-		(pts
-			(xy 179.07 110.49) (xy 180.34 110.49)
-		)
-		(stroke
-			(width 0)
-			(type default)
-		)
-	)
-	(wire
-		(pts
 			(xy 142.24 91.44) (xy 148.59 91.44)
+		)
+		(stroke
+			(width 0)
+			(type default)
+		)
+	)
+	(wire
+		(pts
+			(xy 191.77 105.41) (xy 191.77 104.14)
+		)
+		(stroke
+			(width 0)
+			(type default)
+		)
+	)
+	(wire
+		(pts
+			(xy 190.5 107.95) (xy 191.77 107.95)
 		)
 		(stroke
@@
 		(on_board yes)
 		(dnp no)
-		(fields_autoplaced yes)
 		(property "Reference" "J3"
-			(at 116.84 105.4099 0)
+			(at 113.03 110.49 0)
 			(effects
 				(font
@@
 	(symbol
 		(lib_id "power:+5V")
-		(at 179.07 106.68 0)
+		(at 191.77 104.14 0)
 		(unit 1)
 		(exclude_from_sim no)
@@
 		(dnp no)
 		(property "Reference" "#PWR06"
-			(at 179.07 110.49 0)
+			(at 191.77 107.95 0)
 			(effects
 				(font
@@
 		)
 		(property "Value" "+5V"
-			(at 179.07 102.87 0)
+			(at 191.77 100.33 0)
 			(effects
 				(font
@@
 		)
 		(property "Footprint" ""
-			(at 179.07 106.68 0)
+			(at 191.77 104.14 0)
 			(effects
 				(font
@@
 		)
 		(property "Datasheet" ""
-			(at 179.07 106.68 0)
+			(at 191.77 104.14 0)
 			(effects
 				(font
@@
 		)
 		(property "Description" "Power symbol creates a global label with name \"+5V\""
-			(at 179.07 106.68 0)
+			(at 191.77 104.14 0)
 			(effects
 				(font
@@
 	(symbol
 		(lib_id "power:GND")
-		(at 179.07 111.76 0)
+		(at 191.77 109.22 0)
 		(unit 1)
 		(exclude_from_sim no)
@@
 		(dnp no)
 		(property "Reference" "#PWR07"
-			(at 179.07 118.11 0)
+			(at 191.77 115.57 0)
 			(effects
 				(font
@@
 		)
 		(property "Value" "GND"
-			(at 179.07 115.57 0)
+			(at 191.77 113.03 0)
 			(effects
 				(font
@@
 		)
 		(property "Footprint" ""
-			(at 179.07 111.76 0)
+			(at 191.77 109.22 0)
 			(effects
 				(font
@@
 		)
 		(property "Datasheet" ""
-			(at 179.07 111.76 0)
+			(at 191.77 109.22 0)
 			(effects
 				(font
@@
 		)
 		(property "Description" "Power symbol creates a global label with name \"GND\" , ground"
-			(at 179.07 111.76 0)
+			(at 191.77 109.22 0)
 			(effects
 				(font
@@
 		(dnp no)
 		(property "Reference" "J5"
-			(at 115.57 90.1699 0)
+			(at 112.268 92.964 0)
 			(effects
 				(font
@@
 		(dnp no)
 		(property "Reference" "J1"
-			(at 148.082 86.868 0)
+			(at 147.574 129.032 0)
 			(effects
 				(font
@@
 	(symbol
 		(lib_id "Connector:Screw_Terminal_01x02")
-		(at 185.42 107.95 0)
+		(at 185.42 107.95 180)
 		(unit 1)
 		(exclude_from_sim no)
@@
 		(on_board yes)
 		(dnp no)
-		(fields_autoplaced yes)
 		(property "Reference" "J4"
-			(at 187.96 107.9499 0)
-			(effects
-				(font
-					(size 1.27 1.27)
-				)
-				(justify left)
+			(at 185.674 110.49 0)
+			(effects
+				(font
+					(size 1.27 1.27)
+				)
 			)
 		)
 		(property "Value" "Screw_Terminal_01x02"
-			(at 187.96 110.4899 0)
+			(at 182.88 105.4101 0)
 			(effects
 				(font
@@
 		(dnp no)
 		(property "Reference" "J7"
-			(at 184.15 80.264 0)
-			(effects
-				(font
+			(at 184.15 90.17 0)
+			(effects
+				(font
