File: LedDripStrand/LedDripStrand.kicad_pcb (KiCad board)
At the start: 2 copper layers, 40.6 x 20.3 mm, 9 parts, among them J1 Screw_Terminal_01x02, J2 Conn_01x01_Pin, J3 Screw_Terminal_01x03, J4 Screw_Terminal_01x02

Commit message: incremental updates
Changed lines of the file:
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@@
 			(font
 				(size 1 1)
-				(thickness 0.1)
+				(thickness 0.15)
 			)
 			(justify mirror)
@@
 			(font
 				(size 1 1)
-				(thickness 0.1)
+				(thickness 0.15)
 			)
 		)
 	)
 	(gr_text "+5"
-		(at 133.35 98.425 -90)
+		(at 133.35 98.425 270)
 		(layer "F.SilkS")
 		(effects
 			(font
 				(size 1 1)
-				(thickness 0.1)
+				(thickness 0.15)
 			)
 		)
@@
 			(font
 				(size 1 1)
-				(thickness 0.1)
+				(thickness 0.15)
 			)
 		)
@@
 			(font
 				(size 1 1)
-				(thickness 0.1)
+				(thickness 0.15)
 			)
 		)
@@
 			(font
 				(size 1 1)
-				(thickness 0.1)
+				(thickness 0.15)
 			)
 		)
 	)
 	(gr_text "GND"
-		(at 133.35 104.14 -90)
+		(at 133.35 104.14 270)
 		(layer "F.SilkS")
 		(effects
 			(font
 				(size 1 1)
-				(thickness 0.1)
+				(thickness 0.15)
 			)
 		)
@@
 			(font
 				(size 1 1)
-				(thickness 0.1)
+				(thickness 0.15)
 			)
 		)
@@
 			(font
 				(size 1 1)
-				(thickness 0.1)
+				(thickness 0.15)
 			)
 		)
@@
 			(font
 				(size 1 1)
-				(thickness 0.1)
+				(thickness 0.15)
 			)
 		)
@@
 			(font
 				(size 1 1)
-				(thickness 0.1)
+				(thickness 0.15)
 			)
 		)
@@
 			(font
 				(size 1 1)
-				(thickness 0.1)
+				(thickness 0.15)
 			)
 			(justify left)

Commit message: incremental updates
Parts:
- moved J4 13.0 mm to (162.1, 96.5), turned to -90 degrees
Routing:
- net +5V: track 34.0 -> 31.2 mm
Changed lines of the file:
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@@
 	(footprint "MyTerminalBlock:PHOENIX - TERM BLK 2P SIDE ENT 5.08MM PCB"
 		(layer "F.Cu")
-		(at 170.18 106.68 90)
+		(at 162.066 96.52 -90)
 		(property "Reference" "J4"
 			(at 3.175 -9.135 90)
@@
 		)
 		(property "DigiKey Part" "277-1247-ND"
-			(at 0 0 90)
+			(at 0 0 -90)
 			(unlocked yes)
 			(layer "F.Fab")
@@
 		(attr through_hole)
 		(fp_line
-			(start 10.16 -8.15)
-			(end 0 -8.15)
+			(start 0 0)
+			(end 10.16 0)
+			(stroke
+				(width 0.127)
+				(type solid)
+			)
+			(layer "F.SilkS")
+		)
+		(fp_line
+			(start 10.16 0)
+			(end 10.16 -8.15)
 			(stroke
 				(width 0.127)
@@
 		)
 		(fp_line
-			(start 10.16 0)
-			(end 10.16 -8.15)
+			(start 10.16 -8.15)
+			(end 0 -8.15)
 			(stroke
 				(width 0.127)
@@
 			)
 			(layer "F.SilkS")
+		)
+		(fp_circle
+			(center 2.54 -5.588)
+			(end 2.64 -5.588)
+			(stroke
+				(width 0.2)
+				(type solid)
+			)
+			(fill none)
+			(layer "F.SilkS")
+		)
+		(fp_line
+			(start -0.82 0.25)
+			(end 10.41 0.25)
+			(stroke
+				(width 0.05)
+				(type solid)
+			)
+			(layer "F.CrtYd")
+		)
+		(fp_line
+			(start 10.41 0.25)
+			(end 10.41 -8.4)
+			(stroke
+				(width 0.05)
+				(type solid)
+			)
+			(layer "F.CrtYd")
+		)
+		(fp_line
+			(start -0.82 -8.4)
+			(end -0.82 0.25)
+			(stroke
+				(width 0.05)
+				(type solid)
+			)
+			(layer "F.CrtYd")
+		)
+		(fp_line
+			(start 10.41 -8.4)
+			(end -0.82 -8.4)
+			(stroke
+				(width 0.05)
+				(type solid)
+			)
+			(layer "F.CrtYd")
 		)
 		(fp_line
@@
 				(type solid)
 			)
-			(layer "F.SilkS")
+			(layer "F.Fab")
+		)
+		(fp_line
+			(start 10.16 0)
+			(end 10.16 -8.15)
+			(stroke
+				(width 0.127)
+				(type solid)
+			)
+			(layer "F.Fab")
+		)
+		(fp_line
+			(start 0 -8.15)
+			(end 0 0)
+			(stroke
+				(width 0.127)
+				(type solid)
+			)
+			(layer "F.Fab")
+		)
+		(fp_line
+			(start 10.16 -8.15)
+			(end 0 -8.15)
+			(stroke
+				(width 0.127)
+				(type solid)
+			)
+			(layer "F.Fab")
 		)
 		(fp_circle
@@
 			)
 			(fill none)
-			(layer "F.SilkS")
-		)
-		(fp_line
-			(start 10.41 -8.4)
-			(end -0.82 -8.4)
-			(stroke
-				(width 0.05)
-				(type solid)
-			)
-			(layer "F.CrtYd")
-		)
-		(fp_line
-			(start -0.82 -8.4)
-			(end -0.82 0.25)
-			(stroke
-				(width 0.05)
-				(type solid)
-			)
-			(layer "F.CrtYd")
-		)
-		(fp_line
-			(start 10.41 0.25)
-			(end 10.41 -8.4)
-			(stroke
-				(width 0.05)
-				(type solid)
-			)
-			(layer "F.CrtYd")
-		)
-		(fp_line
-			(start -0.82 0.25)
-			(end 10.41 0.25)
-			(stroke
-				(width 0.05)
-				(type solid)
-			)
-			(layer "F.CrtYd")
-		)
-		(fp_line
-			(start 10.16 -8.15)
-			(end 0 -8.15)
-			(stroke
-				(width 0.127)
-				(type solid)
-			)
-			(layer "F.Fab")
-		)
-		(fp_line
-			(start 0 -8.15)
-			(end 0 0)
-			(stroke
-				(width 0.127)
-				(type solid)
-			)
-			(layer "F.Fab")
-		)
-		(fp_line
-			(start 10.16 0)
-			(end 10.16 -8.15)
-			(stroke
-				(width 0.127)
-				(type solid)
-			)
-			(layer "F.Fab")
-		)
-		(fp_line
-			(start 0 0)
-			(end 10.16 0)
-			(stroke
-				(width 0.127)
-				(type solid)
-			)
-			(layer "F.Fab")
-		)
-		(fp_circle
-			(center 2.54 -5.588)
-			(end 2.64 -5.588)
-			(stroke
-				(width 0.2)
-				(type solid)
-			)
-			(fill none)
 			(layer "F.Fab")
 		)
 		(pad "1" thru_hole rect
-			(at 2.54 -4.05 90)
+			(at 2.54 -4.05 270)
 			(size 1.95 1.95)
 			(drill 1.3)
@@
 		)
 		(pad "2" thru_hole circle
-			(at 7.62 -4.05 90)
+			(at 7.62 -4.05 270)
 			(size 1.95 1.95)
 			(drill 1.3)
@@
 	)
 	(gr_text "GND"
-		(at 171.45 99.06 90)
+		(at 171.45 104.14 90)
 		(layer "F.SilkS")
 		(effects
@@
 	)
 	(gr_text "+5"
-		(at 171.45 104.775 90)
+		(at 171.45 99.06 90)
 		(layer "F.SilkS")
 		(effects
@@
 	)
 	(segment
-		(start 154.446 94.996)
+		(start 138.67 99.06)
+		(end 138.684 99.06)
+		(width 2.54)
+		(layer "F.Cu")
+		(net 2)
+	)
+	(segment
+		(start 138.684 99.06)
+		(end 143.256 94.488)
+		(width 2.54)
+		(layer "F.Cu")
+		(net 2)
+	)
+	(segment
+		(start 158.51 99.06)
 		(end 157.48 98.03)
 		(width 2.54)
@@
 	)
 	(segment
-		(start 140.97 94.996)
-		(end 154.446 94.996)
+		(start 166.116 99.06)
+		(end 158.51 99.06)
 		(width 2.54)
 		(layer "F.Cu")
@@
 	)
 	(segment
-		(start 163.59 104.14)
+		(start 153.938 94.488)
 		(end 157.48 98.03)
 		(width 2.54)
@@
 	)
 	(segment
-		(start 166.13 104.14)
-		(end 163.59 104.14)
+		(start 143.256 94.488)
+		(end 153.938 94.488)
 		(width 2.54)
 		(layer "F.Cu")
-		(net 2)
-	)
-	(segment
-		(start 138.67 97.296)
-		(end 140.97 94.996)
-		(width 2.54)
-		(layer "F.Cu")
-		(net 2)
-	)
-	(segment
-		(start 138.67 99.06)
-		(end 138.67 97.296)
-		(width 2.54)
-		(layer "F.Cu")

Commit message: incremental updates
Parts:
- moved J4 13.0 mm to (170.2, 106.7), turned to 90 degrees
Connections:
- J4 pad 1: +5V -> GND
- J4 pad 2: GND -> +5V
Changed lines of the file:
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@@
 		(property ki_fp_filters "TerminalBlock*:*")
 		(sheetname "Root")
-		(sheetfile "LedStrandDrip.kicad_sch")
+		(sheetfile "LedDripStrand.kicad_sch")
 		(attr through_hole)
 		(fp_line
@@
 		(property ki_fp_filters "Connector*:*_1x??_*")
 		(sheetname "Root")
-		(sheetfile "LedStrandDrip.kicad_sch")
+		(sheetfile "LedDripStrand.kicad_sch")
 		(attr through_hole)
 		(fp_line
@@
 		(property ki_fp_filters "TerminalBlock*:*")
 		(sheetname "Root")
-		(sheetfile "LedStrandDrip.kicad_sch")
+		(sheetfile "LedDripStrand.kicad_sch")
 		(attr through_hole)
 		(fp_line
@@
 	(footprint "MyTerminalBlock:PHOENIX - TERM BLK 2P SIDE ENT 5.08MM PCB"
 		(layer "F.Cu")
-		(at 162.066 96.52 -90)
+		(at 170.18 106.68 90)
 		(property "Reference" "J4"
 			(at 3.175 -9.135 90)
@@
 		)
 		(property "DigiKey Part" "277-1247-ND"
-			(at 0 0 -90)
+			(at 0 0 90)
 			(unlocked yes)
 			(layer "F.Fab")
@@
 		(property ki_fp_filters "TerminalBlock*:*")
 		(sheetname "Root")
-		(sheetfile "LedStrandDrip.kicad_sch")
+		(sheetfile "LedDripStrand.kicad_sch")
 		(attr through_hole)
+		(fp_line
+			(start 10.16 -8.15)
+			(end 0 -8.15)
+			(stroke
+				(width 0.127)
+				(type solid)
+			)
+			(layer "F.SilkS")
+		)
+		(fp_line
+			(start 0 -8.15)
+			(end 0 0)
+			(stroke
+				(width 0.127)
+				(type solid)
+			)
+			(layer "F.SilkS")
+		)
+		(fp_line
+			(start 10.16 0)
+			(end 10.16 -8.15)
+			(stroke
+				(width 0.127)
+				(type solid)
+			)
+			(layer "F.SilkS")
+		)
 		(fp_line
 			(start 0 0)
 			(end 10.16 0)
-			(stroke
-				(width 0.127)
-				(type solid)
-			)
-			(layer "F.SilkS")
-		)
-		(fp_line
-			(start 10.16 0)
-			(end 10.16 -8.15)
-			(stroke
-				(width 0.127)
-				(type solid)
-			)
-			(layer "F.SilkS")
-		)
-		(fp_line
-			(start 0 -8.15)
-			(end 0 0)
-			(stroke
-				(width 0.127)
-				(type solid)
-			)
-			(layer "F.SilkS")
-		)
-		(fp_line
-			(start 10.16 -8.15)
-			(end 0 -8.15)
 			(stroke
 				(width 0.127)
@@
 		)
 		(fp_line
+			(start 10.41 -8.4)
+			(end -0.82 -8.4)
+			(stroke
+				(width 0.05)
+				(type solid)
+			)
+			(layer "F.CrtYd")
+		)
+		(fp_line
+			(start -0.82 -8.4)
+			(end -0.82 0.25)
+			(stroke
+				(width 0.05)
+				(type solid)
+			)
+			(layer "F.CrtYd")
+		)
+		(fp_line
+			(start 10.41 0.25)
+			(end 10.41 -8.4)
+			(stroke
+				(width 0.05)
+				(type solid)
+			)
+			(layer "F.CrtYd")
+		)
+		(fp_line
 			(start -0.82 0.25)
 			(end 10.41 0.25)
@@
 		)
 		(fp_line
-			(start 10.41 0.25)
-			(end 10.41 -8.4)
-			(stroke
-				(width 0.05)
-				(type solid)
-			)
-			(layer "F.CrtYd")
-		)
-		(fp_line
-			(start -0.82 -8.4)
-			(end -0.82 0.25)
-			(stroke
-				(width 0.05)
-				(type solid)
-			)
-			(layer "F.CrtYd")
-		)
-		(fp_line
-			(start 10.41 -8.4)
-			(end -0.82 -8.4)
-			(stroke
-				(width 0.05)
-				(type solid)
-			)
-			(layer "F.CrtYd")
+			(start 10.16 -8.15)
+			(end 0 -8.15)
+			(stroke
+				(width 0.127)
+				(type solid)
+			)
+			(layer "F.Fab")
+		)
+		(fp_line
+			(start 0 -8.15)
+			(end 0 0)
+			(stroke
+				(width 0.127)
+				(type solid)
+			)
+			(layer "F.Fab")
+		)
+		(fp_line
+			(start 10.16 0)
+			(end 10.16 -8.15)
+			(stroke
+				(width 0.127)
+				(type solid)
+			)
+			(layer "F.Fab")
 		)
 		(fp_line
 			(start 0 0)
 			(end 10.16 0)
-			(stroke
-				(width 0.127)
-				(type solid)
-			)
-			(layer "F.Fab")
-		)
-		(fp_line
-			(start 10.16 0)
-			(end 10.16 -8.15)
-			(stroke
-				(width 0.127)
-				(type solid)
-			)
-			(layer "F.Fab")
-		)
-		(fp_line
-			(start 0 -8.15)
-			(end 0 0)
-			(stroke
-				(width 0.127)
-				(type solid)
-			)
-			(layer "F.Fab")
-		)
-		(fp_line
-			(start 10.16 -8.15)
-			(end 0 -8.15)
 			(stroke
 				(width 0.127)
@@
 		)
 		(pad "1" thru_hole rect
-			(at 2.54 -4.05 270)
+			(at 2.54 -4.05 90)
+			(size 1.95 1.95)
+			(drill 1.3)
+			(layers "*.Cu" "*.Mask")
+			(remove_unused_layers no)
+			(net 3 "GND")
+			(pinfunction "Pin_1")
+			(pintype "passive")
+			(solder_mask_margin 0.102)
+		)
+		(pad "2" thru_hole circle
+			(at 7.62 -4.05 90)
 			(size 1.95 1.95)
 			(drill 1.3)
@@
 			(remove_unused_layers no)
 			(net 2 "+5V")
-			(pinfunction "Pin_1")
-			(pintype "passive")
-			(solder_mask_margin 0.102)
-		)
-		(pad "2" thru_hole circle
-			(at 7.62 -4.05 270)
-			(size 1.95 1.95)
-			(drill 1.3)
-			(layers "*.Cu" "*.Mask")
-			(remove_unused_layers no)
-			(net 3 "GND")
 			(pinfunction "Pin_2")
 			(pintype "passive")
@@
 	)
 	(segment
+		(start 166.13 99.06)
+		(end 158.51 99.06)
+		(width 2.54)
+		(layer "F.Cu")
+		(net 2)
+	)
+	(segment
 		(start 138.67 99.06)
 		(end 138.684 99.06)
@@
 		(width 2.54)
 		(layer "F.Cu")
-		(net 2)
-	)
-	(segment
-		(start 166.116 99.06)
-		(end 158.51 99.06)
-		(width 2.54)
-		(layer "F.Cu")
