File: LedDripStrand/LedDripStrand.kicad_sch (KiCad schematic)
At the start: 4 parts, among them J1 Screw_Terminal_01x02, J2 Conn_01x01_Pin, J3 Screw_Terminal_01x03, J4 Screw_Terminal_01x02

Commit message: incremental updates
Connections:
- net +5V: now also J4.2 (Pin_2); no longer J4.1 (Pin_1)
- net GND: now also J4.1 (Pin_1); no longer J4.2 (Pin_2)
Other:
- moved on the sheet: J3, J4
